File: board/buttons.kicad_sch (KiCad schematic)
At the start: 24 parts, among them SW1 SW_Push, SW10 SW_Push, SW11 SW_Push, SW12 SW_Push, SW2 SW_Push, SW3 SW_Push, SW4 SW_Push, SW5 SW_Push, SW6 SW_Push, SW7 SW_Push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

Commit message: tested LCD, button scan and serial output
Parts:
- D1, D10, D11, D12, D2, D3, D4, D5, D6, D7, D8, D9: Farnell Part Number (none) -> 2708389; Manufacturer_Name (none) -> TAIWAN SEMICONDUCTOR; Manufacturer_Part_Number (none) -> TS4148 RYG
- SW1, SW10, SW11, SW12, SW2, SW3, SW4, SW5, SW6, SW7, SW8, SW9: Digi-Key Part Number (none) -> EG1833-ND
Changed lines of the file:
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@@
+      (effects (font (size 1.27 1.27)) hide)
+    )
+    (property "Digi-Key Part Number" "EG1833-ND" (id 4) (at 96.52 74.93 0)
       (effects (font (size 1.27 1.27)) hide)
     )
@@
       (effects (font (size 1.27 1.27)) hide)
     )
+    (property "Digi-Key Part Number" "EG1833-ND" (id 4) (at 186.69 74.93 0)
+      (effects (font (size 1.27 1.27)) hide)
+    )
     (pin "1")
     (pin "2")
@@
       (effects (font (size 1.27 1.27)) hide)
     )
+    (property "Digi-Key Part Number" "EG1833-ND" (id 4) (at 186.69 90.17 0)
+      (effects (font (size 1.27 1.27)) hide)
+    )
     (pin "1")
     (pin "2")
@@
       (effects (font (size 1.27 1.27)) hide)
     )
+    (property "Digi-Key Part Number" "EG1833-ND" (id 4) (at 186.69 107.95 0)
+      (effects (font (size 1.27 1.27)) hide)
+    )
     (pin "1")
     (pin "2")
@@
       (effects (font (size 1.27 1.27)) hide)
     )
+    (property "Farnell Part Number" "2708389" (id 4) (at 105.41 90.17 0)
+      (effects (font (size 1.27 1.27)) hide)
+    )
+    (property "Manufacturer_Name" "TAIWAN SEMICONDUCTOR" (id 5) (at 105.41 90.17 0)
+      (effects (font (size 1.27 1.27)) hide)
+    )
+    (property "Manufacturer_Part_Number" "TS4148 RYG" (id 6) (at 105.41 90.17 0)
+      (effects (font (size 1.27 1.27)) hide)
+    )
     (pin "1")
     (pin "2")
@@
       (effects (font (size 1.27 1.27)) hide)
     )
+    (property "Digi-Key Part Number" "EG1833-ND" (id 4) (at 186.69 125.73 0)
+      (effects (font (size 1.27 1.27)) hide)
+    )
     (pin "1")
     (pin "2")
@@
       (effects (font (size 1.27 1.27)) hide)
     )
+    (property "Digi-Key Part Number" "EG1833-ND" (id 4) (at 143.51 90.17 0)
+      (effects (font (size 1.27 1.27)) hide)
+    )
     (pin "1")
     (pin "2")
@@
       (effects (font (size 1.27 1.27)) hide)
     )
+    (property "Farnell Part Number" "2708389" (id 4) (at 105.41 107.95 0)
+      (effects (font (size 1.27 1.27)) hide)
+    )
+    (property "Manufacturer_Name" "TAIWAN SEMICONDUCTOR" (id 5) (at 105.41 107.95 0)
+      (effects (font (size 1.27 1.27)) hide)
+    )
+    (property "Manufacturer_Part_Number" "TS4148 RYG" (id 6) (at 105.41 107.95 0)
+      (effects (font (size 1.27 1.27)) hide)
+    )
     (pin "1")
     (pin "2")
@@
       (effects (font (size 1.27 1.27)) hide)
     )
+    (property "Farnell Part Number" "2708389" (id 4) (at 152.4 107.95 0)
+      (effects (font (size 1.27 1.27)) hide)
+    )
+    (property "Manufacturer_Name" "TAIWAN SEMICONDUCTOR" (id 5) (at 152.4 107.95 0)
+      (effects (font (size 1.27 1.27)) hide)
+    )
+    (property "Manufacturer_Part_Number" "TS4148 RYG" (id 6) (at 152.4 107.95 0)
+      (effects (font (size 1.27 1.27)) hide)
+    )
     (pin "1")
     (pin "2")
@@
       (effects (font (size 1.27 1.27)) hide)
     )
+    (property "Digi-Key Part Number" "EG1833-ND" (id 4) (at 96.52 107.95 0)
+      (effects (font (size 1.27 1.27)) hide)
+    )
     (pin "1")
     (pin "2")
@@
       (effects (font (size 1.27 1.27)) hide)
     )
+    (property "Digi-Key Part Number" "EG1833-ND" (id 4) (at 143.51 125.73 0)
+      (effects (font (size 1.27 1.27)) hide)
+    )
     (pin "1")
     (pin "2")
@@
       (effects (font (size 1.27 1.27)) hide)
     )
+    (property "Digi-Key Part Number" "EG1833-ND" (id 4) (at 96.52 90.17 0)
+      (effects (font (size 1.27 1.27)) hide)
+    )
     (pin "1")
     (pin "2")
@@
       (effects (font (size 1.27 1.27)) hide)
     )
+    (property "Farnell Part Number" "2708389" (id 4) (at 105.41 125.73 0)
+      (effects (font (size 1.27 1.27)) hide)
+    )
+    (property "Manufacturer_Name" "TAIWAN SEMICONDUCTOR" (id 5) (at 105.41 125.73 0)
+      (effects (font (size 1.27 1.27)) hide)
+    )
+    (property "Manufacturer_Part_Number" "TS4148 RYG" (id 6) (at 105.41 125.73 0)
+      (effects (font (size 1.27 1.27)) hide)
+    )
     (pin "1")
     (pin "2")
@@
       (effects (font (size 1.27 1.27)) hide)
     )
+    (property "Farnell Part Number" "2708389" (id 4) (at 105.41 74.93 0)
+      (effects (font (size 1.27 1.27)) hide)
+    )
+    (property "Manufacturer_Name" "TAIWAN SEMICONDUCTOR" (id 5) (at 105.41 74.93 0)
+      (effects (font (size 1.27 1.27)) hide)
+    )
+    (property "Manufacturer_Part_Number" "TS4148 RYG" (id 6) (at 105.41 74.93 0)
+      (effects (font (size 1.27 1.27)) hide)
+    )
     (pin "1")
     (pin "2")
@@
       (effects (font (size 1.27 1.27)) hide)
     )
+    (property "Farnell Part Number" "2708389" (id 4) (at 152.4 90.17 0)
+      (effects (font (size 1.27 1.27)) hide)
+    )
+    (property "Manufacturer_Name" "TAIWAN SEMICONDUCTOR" (id 5) (at 152.4 90.17 0)
+      (effects (font (size 1.27 1.27)) hide)
+    )
+    (property "Manufacturer_Part_Number" "TS4148 RYG" (id 6) (at 152.4 90.17 0)
+      (effects (font (size 1.27 1.27)) hide)
+    )
     (pin "1")
     (pin "2")
@@
       (effects (font (size 1.27 1.27)) hide)
     )
+    (property "Farnell Part Number" "2708389" (id 4) (at 152.4 74.93 0)
+      (effects (font (size 1.27 1.27)) hide)
+    )
+    (property "Manufacturer_Name" "TAIWAN SEMICONDUCTOR" (id 5) (at 152.4 74.93 0)
+      (effects (font (size 1.27 1.27)) hide)
+    )
+    (property "Manufacturer_Part_Number" "TS4148 RYG" (id 6) (at 152.4 74.93 0)
+      (effects (font (size 1.27 1.27)) hide)
+    )
     (pin "1")
     (pin "2")
@@
       (effects (font (size 1.27 1.27)) hide)
     )
+    (property "Farnell Part Number" "2708389" (id 4) (at 152.4 125.73 0)
+      (effects (font (size 1.27 1.27)) hide)
+    )
+    (property "Manufacturer_Name" "TAIWAN SEMICONDUCTOR" (id 5) (at 152.4 125.73 0)
+      (effects (font (size 1.27 1.27)) hide)
+    )
+    (property "Manufacturer_Part_Number" "TS4148 RYG" (id 6) (at 152.4 125.73 0)
+      (effects (font (size 1.27 1.27)) hide)
+    )
     (pin "1")
     (pin "2")
@@
       (effects (font (size 1.27 1.27)) hide)
     )
+    (property "Digi-Key Part Number" "EG1833-ND" (id 4) (at 143.51 107.95 0)
+      (effects (font (size 1.27 1.27)) hide)
+    )
     (pin "1")
     (pin "2")
@@
       (effects (font (size 1.27 1.27)) hide)
     )
+    (property "Farnell Part Number" "2708389" (id 4) (at 195.58 90.17 0)
+      (effects (font (size 1.27 1.27)) hide)
+    )
+    (property "Manufacturer_Name" "TAIWAN SEMICONDUCTOR" (id 5) (at 195.58 90.17 0)
+      (effects (font (size 1.27 1.27)) hide)
+    )
+    (property "Manufacturer_Part_Number" "TS4148 RYG" (id 6) (at 195.58 90.17 0)
+      (effects (font (size 1.27 1.27)) hide)
+    )
     (pin "1")
     (pin "2")
@@
       (effects (font (size 1.27 1.27)) hide)
     )
+    (property "Farnell Part Number" "2708389" (id 4) (at 195.58 107.95 0)
+      (effects (font (size 1.27 1.27)) hide)
+    )
+    (property "Manufacturer_Name" "TAIWAN SEMICONDUCTOR" (id 5) (at 195.58 107.95 0)
+      (effects (font (size 1.27 1.27)) hide)
+    )
+    (property "Manufacturer_Part_Number" "TS4148 RYG" (id 6) (at 195.58 107.95 0)
+      (effects (font (size 1.27 1.27)) hide)
+    )
     (pin "1")
     (pin "2")
@@
       (effects (font (size 1.27 1.27)) hide)
     )
+    (property "Farnell Part Number" "2708389" (id 4) (at 195.58 74.93 0)
+      (effects (font (size 1.27 1.27)) hide)
+    )
+    (property "Manufacturer_Name" "TAIWAN SEMICONDUCTOR" (id 5) (at 195.58 74.93 0)
+      (effects (font (size 1.27 1.27)) hide)
+    )
+    (property "Manufacturer_Part_Number" "TS4148 RYG" (id 6) (at 195.58 74.93 0)
+      (effects (font (size 1.27 1.27)) hide)
+    )
     (pin "1")
     (pin "2")
@@
       (effects (font (size 1.27 1.27)) hide)
     )
+    (property "Farnell Part Number" "2708389" (id 4) (at 195.58 125.73 0)
+      (effects (font (size 1.27 1.27)) hide)
+    )
+    (property "Manufacturer_Name" "TAIWAN SEMICONDUCTOR" (id 5) (at 195.58 125.73 0)
+      (effects (font (size 1.27 1.27)) hide)
+    )
+    (property "Manufacturer_Part_Number" "TS4148 RYG" (id 6) (at 195.58 125.73 0)
+      (effects (font (size 1.27 1.27)) hide)
+    )
     (pin "1")
     (pin "2")
@@
       (effects (font (size 1.27 1.27)) hide)
     )
+    (property "Digi-Key Part Number" "EG1833-ND" (id 4) (at 96.52 125.73 0)
+      (effects (font (size 1.27 1.27)) hide)
+    )
     (pin "1")
     (pin "2")
@@
       (effects (font (size 1.27 1.27)) hide)
     )
+    (property "Digi-Key Part Number" "EG1833-ND" (id 4) (at 143.51 74.93 0)
+      (effects (font (size 1.27 1.27)) hide)
+    )

Commit message: diode footprint change drom 0805 (2012) to SOD123
Parts:
- D1, D10, D11, D12, D2, D3, D4, D5, D6, D7, D8, D9: footprint Inductor_SMD:L_0805_2012Metric -> Diode_SMD:D_SOD-123
Changed lines of the file:
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@@
       (effects (font (size 1.27 1.27)))
     )
-    (property "Footprint" "Inductor_SMD:L_0805_2012Metric" (at 105.41 90.17 0)
+    (property "Footprint" "Diode_SMD:D_SOD-123" (at 105.41 90.17 0)
       (effects (font (size 1.27 1.27)) hide)
     )
@@
       (effects (font (size 1.27 1.27)))
     )
-    (property "Footprint" "Inductor_SMD:L_0805_2012Metric" (at 105.41 107.95 0)
+    (property "Footprint" "Diode_SMD:D_SOD-123" (at 105.41 107.95 0)
       (effects (font (size 1.27 1.27)) hide)
     )
@@
       (effects (font (size 1.27 1.27)))
     )
-    (property "Footprint" "Inductor_SMD:L_0805_2012Metric" (at 152.4 107.95 0)
+    (property "Footprint" "Diode_SMD:D_SOD-123" (at 152.4 107.95 0)
       (effects (font (size 1.27 1.27)) hide)
     )
@@
       (effects (font (size 1.27 1.27)))
     )
-    (property "Footprint" "Inductor_SMD:L_0805_2012Metric" (at 105.41 125.73 0)
+    (property "Footprint" "Diode_SMD:D_SOD-123" (at 105.41 125.73 0)
       (effects (font (size 1.27 1.27)) hide)
     )
@@
       (effects (font (size 1.27 1.27)))
     )
-    (property "Footprint" "Inductor_SMD:L_0805_2012Metric" (at 105.41 74.93 0)
+    (property "Footprint" "Diode_SMD:D_SOD-123" (at 105.41 74.93 0)
       (effects (font (size 1.27 1.27)) hide)
     )
@@
       (effects (font (size 1.27 1.27)))
     )
-    (property "Footprint" "Inductor_SMD:L_0805_2012Metric" (at 152.4 90.17 0)
+    (property "Footprint" "Diode_SMD:D_SOD-123" (at 152.4 90.17 0)
       (effects (font (size 1.27 1.27)) hide)
     )
@@
       (effects (font (size 1.27 1.27)))
     )
-    (property "Footprint" "Inductor_SMD:L_0805_2012Metric" (at 152.4 74.93 0)
+    (property "Footprint" "Diode_SMD:D_SOD-123" (at 152.4 74.93 0)
       (effects (font (size 1.27 1.27)) hide)
     )
@@
       (effects (font (size 1.27 1.27)))
     )
-    (property "Footprint" "Inductor_SMD:L_0805_2012Metric" (at 152.4 125.73 0)
+    (property "Footprint" "Diode_SMD:D_SOD-123" (at 152.4 125.73 0)
       (effects (font (size 1.27 1.27)) hide)
     )
@@
       (effects (font (size 1.27 1.27)))
     )
-    (property "Footprint" "Inductor_SMD:L_0805_2012Metric" (at 195.58 90.17 0)
+    (property "Footprint" "Diode_SMD:D_SOD-123" (at 195.58 90.17 0)
       (effects (font (size 1.27 1.27)) hide)
     )
@@
       (effects (font (size 1.27 1.27)))
     )
-    (property "Footprint" "Inductor_SMD:L_0805_2012Metric" (at 195.58 107.95 0)
+    (property "Footprint" "Diode_SMD:D_SOD-123" (at 195.58 107.95 0)
       (effects (font (size 1.27 1.27)) hide)
     )
@@
       (effects (font (size 1.27 1.27)))
     )
-    (property "Footprint" "Inductor_SMD:L_0805_2012Metric" (at 195.58 74.93 0)
+    (property "Footprint" "Diode_SMD:D_SOD-123" (at 195.58 74.93 0)
       (effects (font (size 1.27 1.27)) hide)
     )
@@
       (effects (font (size 1.27 1.27)))
     )
-    (property "Footprint" "Inductor_SMD:L_0805_2012Metric" (at 195.58 125.73 0)
-      (effects (font (size 1.27 1.27)) hide)
-    )
+    (property "Footprint" "Diode_SMD:D_SOD-123" (at 195.58 125.73 0)
+      (effects (font (size 1.27 1.27)) hide)
+    )

Commit message: removed software folder
Other:
- title: (none) -> Crane V2.0 Rev A
Changed lines of the file:
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@@
 (kicad_sch (version 20230121) (generator eeschema)
   (paper "A4")
+  (title_block
+    (title "Crane V2.0 Rev A")
+  )
   (junction (at 129.54 107.95) (diameter 0) (color 0 0 0 0)
   )
