File: board/connectors.kicad_sch (KiCad schematic)
At the start: 5 parts, among them J10 Conn_01x05, J11 Conn_01x03, J12 Conn_01x03, J6 292304-1, J8 Conn_ARM_JTAG_SWD_20

Commit message: removed software folder
Other:
- title: (none) -> Crane V2.0 Rev A
Changed lines of the file:
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@@
 (kicad_sch (version 20230121) (generator eeschema)
   (paper "A4")
+  (title_block
+    (title "Crane V2.0 Rev A")
+  )
   (junction (at 77.47 50.8) (diameter 0) (color 0 0 0 0)
   )
