File: board/power.kicad_sch (KiCad schematic)
At the start: 18 parts, among them J11 Conn_01x03_Male, J12 Conn_01x02_Male, J13 Conn_01x02_Male, J14 Conn_01x03_Male, U4 LD3985M33R_SOT23

Commit message: removed software folder
Other:
- title: (none) -> Crane V2.0 Rev A
Changed lines of the file:
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@@
 (kicad_sch (version 20230121) (generator eeschema)
   (paper "A4")
+  (title_block
+    (title "Crane V2.0 Rev A")
+  )
   (junction (at 133.35 161.29) (diameter 0) (color 0 0 0 0)
   )
